Commit message: Add Gazebo Classic spawn for Ackermann vehicle

File: src/ackermann_description/urdf/ackermann_car.urdf.xacro (robot description, xacro)
@@ -217,3 +217,30 @@
     <origin xyz="0.18 0 0.18" rpy="0 0 0"/>
   </joint>
+  <!-- ===================== -->
+  <!-- Gazebo Materials -->
+  <!-- ===================== -->
+  <gazebo reference="base_link">
+    <material>Gazebo/Blue</material>
+  </gazebo>
+  <gazebo reference="front_left_steer_link">
+    <material>Gazebo/Red</material>
+  </gazebo>
+  <gazebo reference="front_right_steer_link">
+    <material>Gazebo/Red</material>
+  </gazebo>
+  <gazebo reference="front_left_wheel_link">
+    <material>Gazebo/Black</material>
+  </gazebo>
+  <gazebo reference="front_right_wheel_link">
+    <material>Gazebo/Black</material>
+  </gazebo>
+  <gazebo reference="rear_left_wheel_link">
+    <material>Gazebo/Black</material>
+  </gazebo>
+  <gazebo reference="rear_right_wheel_link">
+    <material>Gazebo/Black</material>
+  </gazebo>
+  <gazebo reference="laser_link">
+    <material>Gazebo/Grey</material>
+  </gazebo>
 </robot>

Commit message: Add initial ros2 control integration

File: src/ackermann_description/urdf/ackermann_car.urdf.xacro (robot description, xacro)
@@ -218,4 +218,63 @@
   </joint>
   <!-- ===================== -->
+  <!-- ros2_control for Gazebo Classic -->
+  <!-- ===================== -->
+  <ros2_control name="GazeboSystem" type="system">
+    <hardware>
+      <plugin>gazebo_ros2_control/GazeboSystem</plugin>
+    </hardware>
+    <!-- Front steering joints: position command -->
+    <joint name="front_left_steer_joint">
+      <command_interface name="position">
+        <param name="min">-0.6</param>
+        <param name="max">0.6</param>
+      </command_interface>
+      <state_interface name="position"/>
+      <state_interface name="velocity"/>
+    </joint>
+    <joint name="front_right_steer_joint">
+      <command_interface name="position">
+        <param name="min">-0.6</param>
+        <param name="max">0.6</param>
+      </command_interface>
+      <state_interface name="position"/>
+      <state_interface name="velocity"/>
+    </joint>
+    <!-- Front wheel rolling joints: state only for now -->
+    <joint name="front_left_wheel_joint">
+      <state_interface name="position"/>
+      <state_interface name="velocity"/>
+    </joint>
+    <joint name="front_right_wheel_joint">
+      <state_interface name="position"/>
+      <state_interface name="velocity"/>
+    </joint>
+    <!-- Rear traction joints: velocity command -->
+    <joint name="rear_left_wheel_joint">
+      <command_interface name="velocity">
+        <param name="min">-20.0</param>
+        <param name="max">20.0</param>
+      </command_interface>
+      <state_interface name="position"/>
+      <state_interface name="velocity"/>
+    </joint>
+    <joint name="rear_right_wheel_joint">
+      <command_interface name="velocity">
+        <param name="min">-20.0</param>
+        <param name="max">20.0</param>
+      </command_interface>
+      <state_interface name="position"/>
+      <state_interface name="velocity"/>
+    </joint>
+  </ros2_control>
+  <!-- ===================== -->
+  <!-- Gazebo ros2_control Plugin -->
+  <!-- ===================== -->
+  <gazebo>
+    <plugin name="gazebo_ros2_control" filename="libgazebo_ros2_control.so">
+      <parameters>$(find ackermann_control)/config/ros2_control.yaml</parameters>
+    </plugin>
+  </gazebo>
+  <!-- ===================== -->
   <!-- Gazebo Materials -->
   <!-- ===================== -->

Commit message: Add optional ros2_control interfaces to robot model

File: src/ackermann_description/urdf/ackermann_car.urdf.xacro (robot description, xacro)
@@ -1,4 +1,6 @@
 <?xml version="1.0"?>
 <robot name="ackermann_car" xmlns:xacro="http://www.ros.org/wiki/xacro">
+  <xacro:arg name="use_ros2_control" default="false"/>
+  <xacro:arg name="control_config" default=""/>
   <!-- ===================== -->
   <!-- Parameters -->
@@ -244,3 +246,60 @@
     <material>Gazebo/Grey</material>
   </gazebo>
+  <!-- ===================== -->
+  <!-- ros2_control for Gazebo -->
+  <!-- ===================== -->
+  <xacro:if value="$(arg use_ros2_control)">
+    <ros2_control name="GazeboSystem" type="system">
+      <hardware>
+        <plugin>gazebo_ros2_control/GazeboSystem</plugin>
+      </hardware>
+      <joint name="front_left_steer_joint">
+        <command_interface name="position">
+          <param name="min">-0.6</param>
+          <param name="max">0.6</param>
+        </command_interface>
+        <state_interface name="position"/>
+        <state_interface name="velocity"/>
+      </joint>
+      <joint name="front_right_steer_joint">
+        <command_interface name="position">
+          <param name="min">-0.6</param>
+          <param name="max">0.6</param>
+        </command_interface>
+        <state_interface name="position"/>
+        <state_interface name="velocity"/>
+      </joint>
+      <joint name="front_left_wheel_joint">
+        <state_interface name="position"/>
+        <state_interface name="velocity"/>
+      </joint>
+      <joint name="front_right_wheel_joint">
+        <state_interface name="position"/>
+        <state_interface name="velocity"/>
+      </joint>
+      <joint name="rear_left_wheel_joint">
+        <command_interface name="velocity">
+          <param name="min">-20.0</param>
+          <param name="max">20.0</param>
+        </command_interface>
+        <state_interface name="position"/>
+        <state_interface name="velocity"/>
+      </joint>
+      <joint name="rear_right_wheel_joint">
+        <command_interface name="velocity">
+          <param name="min">-20.0</param>
+          <param name="max">20.0</param>
+        </command_interface>
+        <state_interface name="position"/>
+        <state_interface name="velocity"/>
+      </joint>
+    </ros2_control>
+    <gazebo>
+      <plugin name="gazebo_ros2_control" filename="libgazebo_ros2_control.so">
+        <robot_param>robot_description</robot_param>
+        <robot_param_node>robot_state_publisher</robot_param_node>
+        <parameters>$(arg control_config)</parameters>
+      </plugin>
+    </gazebo>
+  </xacro:if>
 </robot>

Commit message: update ackermann simulation model and documentation

File: src/ackermann_description/urdf/ackermann_car.urdf.xacro (robot description, xacro)
@@ -16,4 +16,7 @@
   <xacro:property name="steer_link_length" value="0.04"/>
   <xacro:property name="steer_link_mass"   value="0.10"/>
+  <xacro:property name="laser_radius" value="0.04"/>
+  <xacro:property name="laser_height" value="0.04"/>
+  <xacro:property name="laser_mass"   value="0.10"/>
   <xacro:property name="front_x" value="0.22"/>
   <xacro:property name="rear_x"  value="-0.22"/>
@@ -82,7 +85,13 @@
   <!-- Base Link -->
   <!-- ===================== -->
+  <link name="base_footprint"/>
+  <joint name="base_footprint_joint" type="fixed">
+    <parent link="base_footprint"/>
+    <child link="base_link"/>
+    <origin xyz="0 0 ${wheel_radius + base_height / 2.0}" rpy="0 0 0"/>
+  </joint>
   <link name="base_link">
     <visual>
-      <origin xyz="0 0 ${base_height / 2.0}" rpy="0 0 0"/>
+      <origin xyz="0 0 0" rpy="0 0 0"/>
       <geometry>
         <box size="${base_length} ${base_width} ${base_height}"/>
@@ -90,6 +99,20 @@
       <material name="blue"/>
     </visual>
+    <visual>
+      <origin xyz="${rear_x} 0 ${-base_height / 2.0}" rpy="1.5708 0 0"/>
+      <geometry>
+        <cylinder radius="0.012" length="${left_y - right_y}"/>
+      </geometry>
+      <material name="gray"/>
+    </visual>
+    <visual>
+      <origin xyz="${front_x} 0 ${-base_height / 2.0}" rpy="1.5708 0 0"/>
+      <geometry>
+        <cylinder radius="0.012" length="${left_y - right_y}"/>
+      </geometry>
+      <material name="gray"/>
+    </visual>
     <collision>
-      <origin xyz="0 0 ${base_height / 2.0}" rpy="0 0 0"/>
+      <origin xyz="0 0 0" rpy="0 0 0"/>
       <geometry>
         <box size="${base_length} ${base_width} ${base_height}"/>
@@ -128,5 +151,5 @@
       <parent link="base_link"/>
       <child link="front_${side}_steer_link"/>
-      <origin xyz="${front_x} ${y} ${wheel_radius}" rpy="0 0 0"/>
+      <origin xyz="${front_x} ${y} ${-base_height / 2.0}" rpy="0 0 0"/>
       <axis xyz="0 0 1"/>
       <limit lower="-0.6" upper="0.6" effort="10.0" velocity="2.0"/>
@@ -184,5 +207,5 @@
       <parent link="base_link"/>
       <child link="rear_${side}_wheel_link"/>
-      <origin xyz="${rear_x} ${y} ${wheel_radius}" rpy="0 0 0"/>
+      <origin xyz="${rear_x} ${y} ${-base_height / 2.0}" rpy="0 0 0"/>
       <axis xyz="0 1 0"/>
     </joint>
@@ -202,5 +225,5 @@
       <origin xyz="0 0 0" rpy="0 0 0"/>
       <geometry>
-        <cylinder radius="0.04" length="0.04"/>
+        <cylinder radius="${laser_radius}" length="${laser_height}"/>
       </geometry>
       <material name="gray"/>
@@ -209,13 +232,13 @@
       <origin xyz="0 0 0" rpy="0 0 0"/>
       <geometry>
-        <cylinder radius="0.04" length="0.04"/>
+        <cylinder radius="${laser_radius}" length="${laser_height}"/>
       </geometry>
     </collision>
-    <xacro:cylinder_inertia_z_axis m="0.1" r="0.04" l="0.04"/>
+    <xacro:cylinder_inertia_z_axis m="${laser_mass}" r="${laser_radius}" l="${laser_height}"/>
   </link>
   <joint name="laser_joint" type="fixed">
     <parent link="base_link"/>
     <child link="laser_link"/>
-    <origin xyz="0.18 0 0.18" rpy="0 0 0"/>
+    <origin xyz="0.18 0 ${base_height / 2.0 + laser_height / 2.0}" rpy="0 0 0"/>
   </joint>
   <!-- ===================== -->
